Commit message: migrate to gazebo_ignition

File: Software/ROS2_Env/kr3r540_ws/src/kr3r540_description/urdf/kr3r540.urdf.xacro (robot description, xacro)
@@ -1,221 +1,224 @@
 <?xml version="1.0"?>
 <robot xmlns:xacro="http://wiki.ros.org/xacro" name="kr3r540">
- 	    <xacro:include filename="kr3r540_gazebo.xacro" />
-      <xacro:include filename="kr3r540_ros2_control.xacro"/>
-  <!-- Define Links -->
-  <link name="world_link">
-  </link>
-  <link name="base_link">
-    <visual>
-      <geometry>
-        <mesh filename="package://kr3r540_description/meshes/visual/base_link.stl"/>
-      </geometry>
-      <material name="kuka_pedestal">
-        <color rgba="0.50588 0.47059 0.38824 1.0"/>
-      </material>
-    </visual>
-    <collision>
-      <geometry>
-        <mesh filename="package://kr3r540_description/meshes/collision/base_link.stl"/>
-      </geometry>
-    </collision>
-    <inertial>
-      <origin xyz="0 0 0" rpy="0 0 0"/>
-      <mass value="11.37"/>
-      <inertia ixx="0.537" ixy="0.002" ixz="0.014" iyy="0.804" iyz="0.00" izz="0.745"/>
-    </inertial>
-  </link>
-  <link name="link_1">
-    <visual>
-      <geometry>
-        <mesh filename="package://kr3r540_description/meshes/visual/link_1.stl"/>
-      </geometry>
-      <material name="kuka_ral_pure_white">
-        <color rgba="1.0 1.0 1.0 1.0"/>
-      </material>
-    </visual>
-    <collision>
-      <geometry>
-        <mesh filename="package://kr3r540_description/meshes/collision/link_1.stl"/>
-      </geometry>
-    </collision>
-    <inertial>
-      <origin xyz="0 0 0" rpy="0 0 0"/>
-      <mass value="7"/>
-      <inertia ixx="0.361" ixy="-0.001" ixz="-0.0014" iyy="0.255" iyz="-0.007" izz="0.29"/>
-    </inertial>
-  </link>
-  <link name="link_2">
-    <visual>
-      <geometry>
-        <mesh filename="package://kr3r540_description/meshes/visual/link_2.stl"/>
-      </geometry>
-      <material name="kuka_ral_pure_white">
-        <color rgba="1.0 1.0 1.0 1.0"/>
-      </material>
-    </visual>
-    <collision>
-      <geometry>
-        <mesh filename="package://kr3r540_description/meshes/collision/link_2.stl"/>
-      </geometry>
-    </collision>
-    <inertial>
-      <origin xyz="0 0 0" rpy="0 0 0"/>
-      <mass value="6.9"/>
-      <inertia ixx="0.249" ixy="-0.007" ixz="-0.021" iyy="0.573" iyz="-0.001" izz="0.708"/>
-    </inertial>
-  </link>
-  <link name="link_3">
-    <visual>
-      <geometry>
-        <mesh filename="package://kr3r540_description/meshes/visual/link_3.stl"/>
-      </geometry>
-      <material name="kuka_ral_pure_white">
-        <color rgba="1.0 1.0 1.0 1.0"/>
-      </material>
-    </visual>
-    <collision>
-      <geometry>
-        <mesh filename="package://kr3r540_description/meshes/collision/link_3.stl"/>
-      </geometry>
-    </collision>
-    <inertial>
-      <origin xyz="0 0 0" rpy="0 0 0"/>
-      <mass value="3"/>
-      <inertia ixx="0.05" ixy="0.00" ixz="-0.009" iyy="0.09" iyz="3.291" izz="0.085"/>
-    </inertial>
-  </link>
-  <link name="link_4">
-    <visual>
-      <geometry>
-        <mesh filename="package://kr3r540_description/meshes/visual/link_4.stl"/>
-      </geometry>
-      <material name="kuka_ral_pure_white">
-        <color rgba="1.0 1.0 1.0 1.0"/>
-      </material>
-    </visual>
-    <collision>
-      <geometry>
-        <mesh filename="package://kr3r540_description/meshes/collision/link_4.stl"/>
-      </geometry>
-    </collision>
-    <inertial>
-      <origin xyz="0 0 0" rpy="0 0 0"/>
-      <mass value="2"/>
-      <inertia ixx="0.04" ixy="-0.004" ixz="0.00" iyy="0.045" iyz="-0.001" izz="0.063"/>
-    </inertial>
-  </link>
-  <link name="link_5">
-    <visual>
-      <geometry>
-        <mesh filename="package://kr3r540_description/meshes/visual/link_5.stl"/>
-      </geometry>
-      <material name="kuka_ral_pure_white">
-        <color rgba="1.0 1.0 1.0 1.0"/>
-      </material>
-    </visual>
-    <collision>
-      <geometry>
-        <mesh filename="package://kr3r540_description/meshes/collision/link_5.stl"/>
-      </geometry>
-    </collision>
-    <inertial>
-      <origin xyz="0 0 0" rpy="0 0 0"/>
-      <mass value="1"/>
-      <inertia ixx="0.009" ixy="0.00" ixz="-9.12" iyy="0.012" iyz="8.691" izz="0.014"/>
-    </inertial>
-  </link>
-  <link name="link_6">
-    <visual>
-      <geometry>
-        <mesh filename="package://kr3r540_description/meshes/visual/link_6.stl"/>
-      </geometry>
-      <material name="kuka_pedestal">
-        <color rgba="0.50588 0.47059 0.38824 1.0"/>
-      </material>
-    </visual>
-    <collision>
-      <geometry>
-        <mesh filename="package://kr3r540_description/meshes/collision/link_6.stl"/>
-      </geometry>
-    </collision>
-    <inertial>
-      <origin xyz="0 0 0" rpy="0 0 0"/>
-      <mass value="0.03"/>
-      <inertia ixx="9.585" ixy="-6.57" ixz="-2.07" iyy="5.139" iyz="-7.11" izz="5.14"/>
-    </inertial>
-  </link>
-  <link name="greifer">
-    <visual>
-      <geometry>
-        <mesh filename="package://kr3r540_description/meshes/visual/greifer.stl" scale="0.1 0.1 0.1"/>
-      </geometry>
-      <material name="kuka_black">
-        <color rgba="0.0549 0.0549 0.0627 1.0"/>
-      </material>
-    </visual>
-    <collision>
-      <geometry>
-        <mesh filename="package://kr3r540_description/meshes/collision/greifer.stl" scale="0.1 0.1 0.1"/>
-      </geometry>
-    </collision>
-    <inertial>
-      <origin xyz="0 0 0" rpy="0 0 0"/>
-      <mass value="0.19"/>
-      <inertia ixx="13.106" ixy="-0.034" ixz="0.083" iyy="14.078" iyz="0.17" izz="4.086"/>
-    </inertial>
-  </link>
-  <!-- Define Joints -->
-  <joint name="world_to_base" type="fixed">
-    <parent link="world_link"/>
-    <child link="base_link"/>
-    <origin xyz="0 0 0" rpy="0 0 0"/>
-  </joint>
-  <joint name="joint_1" type="revolute">
-    <parent link="base_link"/>
-    <child link="link_1"/>
-    <origin xyz="0 0 0.345" rpy="0 0 0"/>
-    <axis xyz="0 0 -1"/>
-    <limit lower="-2.967" upper="2.967" effort="0" velocity="9.266"/>
-  </joint>
-  <joint name="joint_2" type="revolute">
-    <parent link="link_1"/>
-    <child link="link_2"/>
-    <origin xyz="0.020 0 0" rpy="0 0 0"/>
-    <axis xyz="0 1 0"/>
-    <limit lower="-2.967" upper="0.872665" effort="0" velocity="9.233"/>
-  </joint>
-  <joint name="joint_3" type="revolute">
-    <parent link="link_2"/>
-    <child link="link_3"/>
-    <origin xyz="0.260 0 0" rpy="0 0 0"/>
-    <axis xyz="0 1 0"/>
-    <limit lower="-1.919" upper="2.705" effort="0" velocity="9.389"/>
-  </joint>
-  <joint name="joint_4" type="revolute">
-    <parent link="link_3"/>
-    <child link="link_4"/>
-    <origin xyz="0 0 0.020" rpy="0 0 0"/>
-    <axis xyz="-1 0 0"/>
-    <limit lower="-3.054" upper="3.054" effort="0" velocity="10.472"/>
-  </joint>
-  <joint name="joint_5" type="revolute">
-    <parent link="link_4"/>
-    <child link="link_5"/>
-     <origin xyz="0.260 0 0" rpy="0 0 0"/>
-    <axis xyz="0 1 0"/>
-    <limit lower="-2.094" upper="2.094" effort="0" velocity="10.472"/>
-  </joint>
-  <joint name="joint_6" type="revolute">
-    <parent link="link_5"/>
-    <child link="link_6"/>
-    <origin xyz="0.075 0 0" rpy="0 0 0"/>
-    <axis xyz="-1 0 0"/>
-    <limit lower="-6.108" upper="6.108" effort="0" velocity="13.962"/>
-  </joint>
-  <joint name="flange" type="fixed">
-    <parent link="link_6"/>
-    <child link="greifer"/>
-    <origin xyz="0.032 0 -0.02" rpy="0 0 1.5708"/>
-  </joint>
+ 	    <!-- xacro:include filename="kr3r540_gazebo.xacro" -->
+      <!-- xacro:include filename="kr3r540_ros2_control.xacro" -->
+ <!-- Define Links -->
+ <link name="world_link">
+</link>
+<link name="base_link">
+  <visual>
+    <geometry>
+      <mesh filename="package://kr3r540_description/meshes/visual/base_link.stl"/>
+    </geometry>
+    <material name="kuka_pedestal">
+      <color rgba="0.50588 0.47059 0.38824 1.0"/>
+    </material>
+  </visual>
+  <collision>
+    <geometry>
+      <mesh filename="package://kr3r540_description/meshes/collision/base_link.stl"/>
+    </geometry>
+  </collision>
+  <inertial>
+    <origin xyz="0 0 0" rpy="0 0 0"/>
+    <mass value="11.37"/>
+    <inertia ixx="0.537" ixy="0.002" ixz="0.014" iyy="0.804" iyz="0.00" izz="0.745"/>
+  </inertial>
+</link>
+<link name="link_1">
+  <visual>
+    <geometry>
+      <mesh filename="package://kr3r540_description/meshes/visual/link_1.stl"/>
+    </geometry>
+    <material name="kuka_ral_pure_white">
+      <color rgba="1.0 1.0 1.0 1.0"/>
+    </material>
+  </visual>
+  <collision>
+    <geometry>
+      <mesh filename="package://kr3r540_description/meshes/collision/link_1.stl"/>
+    </geometry>
+  </collision>
+  <inertial>
+    <origin xyz="0 0 0" rpy="0 0 0"/>
+    <mass value="7"/>
+    <inertia ixx="0.361" ixy="-0.001" ixz="-0.0014" iyy="0.255" iyz="-0.007" izz="0.29"/>
+  </inertial>
+</link>
+<link name="link_2">
+  <visual>
+    <geometry>
+      <mesh filename="package://kr3r540_description/meshes/visual/link_2.stl"/>
+    </geometry>
+    <material name="kuka_ral_pure_white">
+      <color rgba="1.0 1.0 1.0 1.0"/>
+    </material>
+  </visual>
+  <collision>
+    <geometry>
+      <mesh filename="package://kr3r540_description/meshes/collision/link_2.stl"/>
+    </geometry>
+  </collision>
+  <inertial>
+    <origin xyz="0 0 0" rpy="0 0 0"/>
+    <mass value="6.9"/>
+    <inertia ixx="0.249" ixy="-0.007" ixz="-0.021" iyy="0.573" iyz="-0.001" izz="0.708"/>
+  </inertial>
+</link>
+<link name="link_3">
+  <visual>
+    <geometry>
+      <mesh filename="package://kr3r540_description/meshes/visual/link_3.stl"/>
+    </geometry>
+    <material name="kuka_ral_pure_white">
+      <color rgba="1.0 1.0 1.0 1.0"/>
+    </material>
+  </visual>
+  <collision>
+    <geometry>
+      <mesh filename="package://kr3r540_description/meshes/collision/link_3.stl"/>
+    </geometry>
+  </collision>
+  <inertial>
+    <origin xyz="0 0 0" rpy="0 0 0"/>
+    <mass value="3"/>
+    <inertia ixx="0.005464170195346057" ixy="2.317865761359266e-05" ixz="-0.0008376172568479034"
+            iyy="0.009668497673794239" iyz="-5.3812765981131285e-06" izz="0.009530838326239676"/>
+</inertial>
+</link>
+<link name="link_4">
+  <visual>
+    <geometry>
+      <mesh filename="package://kr3r540_description/meshes/visual/link_4.stl"/>
+    </geometry>
+    <material name="kuka_ral_pure_white">
+      <color rgba="1.0 1.0 1.0 1.0"/>
+    </material>
+  </visual>
+  <collision>
+    <geometry>
+      <mesh filename="package://kr3r540_description/meshes/collision/link_4.stl"/>
+    </geometry>
+  </collision>
+  <inertial>
+    <origin xyz="0 0 0" rpy="0 0 0"/>
+    <mass value="2"/>
+    <inertia ixx="0.04" ixy="-0.004" ixz="0.00" iyy="0.045" iyz="-0.001" izz="0.063"/>
+  </inertial>
+</link>
+<link name="link_5">
+  <visual>
+    <geometry>
+      <mesh filename="package://kr3r540_description/meshes/visual/link_5.stl"/>
+    </geometry>
+    <material name="kuka_ral_pure_white">
+      <color rgba="1.0 1.0 1.0 1.0"/>
+    </material>
+  </visual>
+  <collision>
+    <geometry>
+      <mesh filename="package://kr3r540_description/meshes/collision/link_5.stl"/>
+    </geometry>
+  </collision>
+  <inertial>
+    <origin xyz="0 0 0" rpy="0 0 0"/>
+    <mass value="1"/>
+    <inertia ixx="0.0009523921025026232" ixy="-1.4859377039896955e-05" ixz="-2.6599547296907754e-07"
+            iyy="0.001277581091791774" iyz="2.9443366764204974e-07" izz="0.0014178861490860182"/>
+</inertial>
+</link>
+<link name="link_6">
+  <visual>
+    <geometry>
+      <mesh filename="package://kr3r540_description/meshes/visual/link_6.stl"/>
+    </geometry>
+    <material name="kuka_pedestal">
+      <color rgba="0.50588 0.47059 0.38824 1.0"/>
+    </material>
+  </visual>
+  <collision>
+    <geometry>
+      <mesh filename="package://kr3r540_description/meshes/collision/link_6.stl"/>
+    </geometry>
+  </collision>
+  <inertial>
+    <origin xyz="0 0 0" rpy="0 0 0"/>
+    <mass value="0.03"/>
+    <inertia ixx="9.7510332695528e-06" ixy="-5.535554975934552e-11" ixz="1.0491860620923319e-16"
+            iyy="5.458075446678377e-06" iyz="-3.0083248575603903e-19" izz="5.45822894382603e-06"/>
+</inertial>
+</link>
+<link name="greifer">
+  <visual>
+    <geometry>
+      <mesh filename="package://kr3r540_description/meshes/visual/greifer.stl" scale="0.1 0.1 0.1"/>
+    </geometry>
+    <material name="kuka_black">
+      <color rgba="0.0549 0.0549 0.0627 1.0"/>
+    </material>
+  </visual>
+  <collision>
+    <geometry>
+      <mesh filename="package://kr3r540_description/meshes/collision/greifer.stl" scale="0.1 0.1 0.1"/>
+    </geometry>
+  </collision>
+  <inertial>
+    <origin xyz="0 0 0" rpy="0 0 0"/>
+    <mass value="0.19"/>
+    <inertia ixx="13.106" ixy="-0.034" ixz="0.083" iyy="14.078" iyz="0.17" izz="4.086"/>
+  </inertial>
+</link>
+<!-- Define Joints -->
+<joint name="world_to_base" type="fixed">
+  <parent link="world_link"/>
+  <child link="base_link"/>
+  <origin xyz="0 0 0" rpy="0 0 0"/>
+</joint>
+<joint name="joint_1" type="revolute">
+  <parent link="base_link"/>
+  <child link="link_1"/>
+  <origin xyz="0 0 0.345" rpy="0 0 0"/>
+  <axis xyz="0 0 -1"/>
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
File: Software/ROS2_Env/kr3r540_ws/src/kr3r540_description/urdf/kr3r540_ros2_control.xacro (robot description, xacro)
@@ -1,4 +1,9 @@
 <?xml version="1.0" encoding="UTF-8"?>
 <robot xmlns:xacro="http://www.ros.org/wiki/xacro">
+    <gazebo>
+        <plugin name="gazebo_ros2_control" filename="libgazebo_ros2_control.so">
+            <parameters>$(find kr3r540_bringup)/sim_config/kr3r540_sim_controllers.yaml</parameters>
+        </plugin>
+    </gazebo>
     <!-- Define PI -->
     <xacro:property name="PI" value="3.14159"/>
@@ -51,9 +56,3 @@
         </joint>
     </ros2_control>
-    <gazebo>
-        <plugin name="gazebo_ros2_control" filename="libgazebo_ros2_control.so">
-            <robot_namespace>kr3r540_sim</robot_namespace>
-          <robot_param>robot_description</robot_param>
-        </plugin>
-    </gazebo>
 </robot>

Commit message: update : ros2 control is running

File: Software/ROS2_Env/kr3r540_ws/src/kr3r540_description/urdf/kr3r540.urdf.xacro (robot description, xacro)
@@ -1,7 +1,4 @@
 <?xml version="1.0"?>
 <robot xmlns:xacro="http://wiki.ros.org/xacro" name="kr3r540">
- 	    <!-- xacro:include filename="kr3r540_gazebo.xacro" -->
-      <!-- xacro:include filename="kr3r540_ros2_control.xacro" -->
- <!-- Define Links -->
  <link name="world_link">
 </link>
@@ -222,3 +219,5 @@
   <origin xyz="0.032 0 -0.02" rpy="0 0 1.5708"/>
 </joint>
+<xacro:include filename="kr3r540_gazebo.xacro"/>
+<xacro:include filename="kr3r540_ros2_control.xacro"/>
 </robot>

File: Software/ROS2_Env/kr3r540_ws/src/kr3r540_description/urdf/kr3r540_gazebo.xacro (robot description, xacro)
@@ -1,27 +1,32 @@
-<?xml version="1.0"?>
-<robot xmlns:xacro="http://www.ros.org/wiki/xacro" name="kr3r540">
+<?xml version="1.0" encoding="UTF-8"?>
+<robot xmlns:xacro="http://www.ros.org/wiki/xacro">
+    <gazebo>
+        <plugin filename="libign_ros2_control-system.so" name="ign_ros2_control::IgnitionROS2ControlPlugin">
+            <parameters>$(find kr3r540_bringup)/sim_config/kr3r540_sim_controllers.yaml</parameters>
+        </plugin>
+    </gazebo>
     <gazebo reference="base_link">
-        <material>Gazebo/Grey</material>
-    </gazebo>
-    <gazebo reference="link_1">
+        <material>Gazebo/Red</material>
+      </gazebo>
+      <gazebo reference="link_1">
          <material>Gazebo/White</material>
-    </gazebo>
-    <gazebo reference="link_2">
+      </gazebo>
+      <gazebo reference="link_2">
          <material>Gazebo/White</material>
-    </gazebo>
-    <gazebo reference="link_3">
+      </gazebo>
+      <gazebo reference="link_3">
          <material>Gazebo/White</material>
-    </gazebo>
-     <gazebo reference="link_4">
+      </gazebo>
+      <gazebo reference="link_4">
          <material>Gazebo/White</material>
-    </gazebo>
-    <gazebo reference="link_5">
+      </gazebo>
+      <gazebo reference="link_5">
          <material>Gazebo/White</material>
-    </gazebo>
-    <gazebo reference="link_6">
+      </gazebo>
+      <gazebo reference="link_6">
         <material>Gazebo/White</material>
-    </gazebo>
-     <gazebo reference="greifer">
+      </gazebo>
+      <gazebo reference="greifer">
          <material>Gazebo/DarkGrey</material>
-    </gazebo>
+      </gazebo>
 </robot>

File: Software/ROS2_Env/kr3r540_ws/src/kr3r540_description/urdf/kr3r540_ros2_control.xacro (robot description, xacro)
@@ -1,18 +1,12 @@
 <?xml version="1.0" encoding="UTF-8"?>
 <robot xmlns:xacro="http://www.ros.org/wiki/xacro">
-    <gazebo>
-        <plugin name="gazebo_ros2_control" filename="libgazebo_ros2_control.so">
-            <parameters>$(find kr3r540_bringup)/sim_config/kr3r540_sim_controllers.yaml</parameters>
-        </plugin>
-    </gazebo>
-    <!-- Define PI -->
     <xacro:property name="PI" value="3.14159"/>
     <ros2_control name="kr3r540_sim_robot" type="system">
         <hardware>
-            <plugin>gazebo_ros2_control/GazeboSystem</plugin>
+            <plugin>ign_ros2_control/IgnitionSystem</plugin>
         </hardware>
         <!-- Define all joints with position interfaces using formula directly -->
         <joint name="joint_1">
-            <command_interface name="position">
+            <command_interface name="position" initial_value="${PI/2}">
                 <param name="min_position">${-170 * PI / 180}</param>
                 <param name="max_position">${170 * PI / 180}</param>

Commit message: testing controller

File: Software/ROS2_Env/kr3r540_ws/src/kr3r540_description/urdf/kr3r540.urdf.xacro (robot description, xacro)
@@ -179,5 +179,5 @@
   <origin xyz="0 0 0.345" rpy="0 0 0"/>
   <axis xyz="0 0 -1"/>
-  <limit lower="-2.967" upper="2.967" effort="0" velocity="9.266"/>
+  <limit lower="-2.967" upper="2.967" effort="1000" velocity="9.266"/>
 </joint>
 <joint name="joint_2" type="revolute">
@@ -186,5 +186,5 @@
   <origin xyz="0.020 0 0" rpy="0 0 0"/>
   <axis xyz="0 1 0"/>
-  <limit lower="-2.967" upper="0.872665" effort="0" velocity="9.233"/>
+  <limit lower="-2.967" upper="0.872665" effort="1000" velocity="9.233"/>
 </joint>
 <joint name="joint_3" type="revolute">
@@ -193,5 +193,5 @@
   <origin xyz="0.260 0 0" rpy="0 0 0"/>
   <axis xyz="0 1 0"/>
-  <limit lower="-1.919" upper="2.705" effort="0" velocity="9.389"/>
+  <limit lower="-1.919" upper="2.705" effort="1000" velocity="9.389"/>
 </joint>
 <joint name="joint_4" type="revolute">
@@ -200,5 +200,5 @@
   <origin xyz="0 0 0.020" rpy="0 0 0"/>
   <axis xyz="-1 0 0"/>
-  <limit lower="-3.054" upper="3.054" effort="0" velocity="10.472"/>
+  <limit lower="-3.054" upper="3.054" effort="1000" velocity="10.472"/>
 </joint>
 <joint name="joint_5" type="revolute">
@@ -207,5 +207,5 @@
    <origin xyz="0.260 0 0" rpy="0 0 0"/>
   <axis xyz="0 1 0"/>
-  <limit lower="-2.094" upper="2.094" effort="0" velocity="10.472"/>
+  <limit lower="-2.094" upper="2.094" effort="1000" velocity="10.472"/>
 </joint>
 <joint name="joint_6" type="revolute">
@@ -214,5 +214,5 @@
   <origin xyz="0.075 0 0" rpy="0 0 0"/>
   <axis xyz="-1 0 0"/>
-  <limit lower="-6.108" upper="6.108" effort="0" velocity="13.962"/>
+  <limit lower="-6.108" upper="6.108" effort="1000" velocity="13.962"/>
 </joint>
 <joint name="flange" type="fixed">

File: Software/ROS2_Env/kr3r540_ws/src/kr3r540_description/urdf/kr3r540_ros2_control.xacro (robot description, xacro)
@@ -1,4 +1,6 @@
 <?xml version="1.0" encoding="UTF-8"?>
 <robot xmlns:xacro="http://www.ros.org/wiki/xacro" name="kr3r540">
+    <xacro:property name="yaml_file_path" value="$(find kr3r540_bringup)/sim_config/initial_positions_sim.yaml"/>
+    <xacro:property name="initial_positions" value="${xacro.load_yaml(yaml_file_path)}"/>
     <xacro:property name="PI" value="3.14159"/>
     <ros2_control name="kr3r540_sim_robot" type="system">
@@ -8,9 +10,12 @@
         <!-- Define all joints with position interfaces using formula directly -->
         <joint name="joint_1">
-            <command_interface name="position">
+            <command_interface name="position" >
                 <param name="min">${-170 * PI / 180}</param>
                 <param name="max">${170 * PI / 180}</param>
             </command_interface>
-            <state_interface name="position"/>
+            <state_interface name="position">
+                <param name="initial_value">${initial_positions.initial_positions.joint_1}</param>
+            </state_interface>
+            <state_interface name="velocity"/>
         </joint>
         <joint name="joint_2">
@@ -19,5 +24,8 @@
                 <param name="max">${50 * PI / 180}</param>
             </command_interface>
-            <state_interface name="position"/>
+            <state_interface name="position">
+                <param name="initial_value">${initial_positions.initial_positions.joint_2}</param>
+            </state_interface>
+            <state_interface name="velocity"/>
         </joint>
         <joint name="joint_3">
@@ -26,5 +34,8 @@
                 <param name="max">${155 * PI / 180}</param>
             </command_interface>
-            <state_interface name="position"/>
+            <state_interface name="position">
+                <param name="initial_value">${initial_positions.initial_positions.joint_3}</param>
+            </state_interface>
+            <state_interface name="velocity"/>
         </joint>
         <joint name="joint_4">
@@ -33,5 +44,8 @@
                 <param name="max">${175 * PI / 180}</param>
             </command_interface>
-            <state_interface name="position"/>
+            <state_interface name="position">
+                <param name="initial_value">${initial_positions.initial_positions.joint_4}</param>
+            </state_interface>
+            <state_interface name="velocity"/>
         </joint>
         <joint name="joint_5">
@@ -40,5 +54,8 @@
                 <param name="max">${120 * PI / 180}</param>
             </command_interface>
-            <state_interface name="position"/>
+            <state_interface name="position">
+                <param name="initial_value">${initial_positions.initial_positions.joint_5}</param>
+            </state_interface>
+            <state_interface name="velocity"/>
         </joint>
         <joint name="joint_6">
@@ -47,5 +64,8 @@
                 <param name="max">${350 * PI / 180}</param>
             </command_interface>
-            <state_interface name="position"/>
+            <state_interface name="position">
+                <param name="initial_value">${initial_positions.initial_positions.joint_6}</param>
+            </state_interface>
+            <state_interface name="velocity"/>
         </joint>
     </ros2_control>
