Commit message: update : added new library for myaxis variable

File: Software/ROS2_Env/kr3r540_ws/src/kr3r540_description/urdf/kr3r540.urdf.xacro (robot description, xacro)
@@ -3,5 +3,5 @@
 <xacro:include filename="kr3r540_gazebo.xacro"/>
 <xacro:include filename="kr3r540_ros2_control.xacro"/>
- <link name="world_link">
+ <link name="world">
 </link>
 <link name="base_link">
@@ -170,5 +170,5 @@
 <!-- Define Joints -->
 <joint name="world_to_base" type="fixed">
-  <parent link="world_link"/>
+  <parent link="world"/>
   <child link="base_link"/>
   <origin xyz="0 0 0" rpy="0 0 0"/>

Commit message: update : added a new ros2 package to handle the digital twin also we need to figure out the (information path ) form sim to real with a usecase

File: Software/ROS2_Env/kr3r540_ws/src/kr3r540_description/urdf/kr3r540.urdf.xacro (robot description, xacro)
@@ -220,5 +220,5 @@
   <parent link="link_6"/>
   <child link="greifer"/>
-  <origin xyz="0.032 0 -0.02" rpy="0 0 1.5708"/>
+  <origin xyz="0.032 0 0.02" rpy="0 ${2*1.5708} 1.5708"/>
 </joint>
 </robot>

Commit message: added : Gripper functionally (Bugged)

File: Software/ROS2_Env/kr3r540_ws/src/kr3r540_description/urdf/kr3r540.urdf.xacro (robot description, xacro)
@@ -149,8 +149,8 @@
 </inertial>
 </link>
-<link name="greifer">
-  <visual>
-    <geometry>
-      <mesh filename="package://kr3r540_description/meshes/visual/greifer.stl" scale="0.1 0.1 0.1"/>
+<link name="greifer_base">
+  <visual>
+    <geometry>
+      <mesh filename="package://kr3r540_description/meshes/visual/Base_visual.stl" scale="0.001 0.001 0.001"/>
     </geometry>
     <material name="kuka_black">
@@ -160,4 +160,66 @@
   <collision>
     <geometry>
+      <mesh filename="package://kr3r540_description/meshes/collision/Base_collusion.stl" scale="0.001 0.001 0.001"/>
+    </geometry>
+  </collision>
+  <inertial>
+    <origin xyz="0 0 0" rpy="0 0 0"/>
+    <mass value="0.19"/>
+    <inertia ixx="0.008552" ixy="-0.000097" ixz="0"
+            iyy="0.002908" iyz="0.000004" izz="0.009732"/>
+  </inertial>
+</link>
+<link name="greifer_finger_1">
+  <visual>
+    <geometry>
+      <mesh filename="package://kr3r540_description/meshes/visual/Finger_1_visual.stl" scale="0.001 0.001 0.001"/>
+    </geometry>
+    <material name="kuka_pedestal">
+      <color rgba="0.50588 0.47059 0.38824 1.0"/>
+    </material>
+  </visual>
+  <collision>
+    <geometry>
+      <mesh filename="package://kr3r540_description/meshes/collision/Finger_1_collusion.stl" scale="0.001 0.001 0.001"/>
+    </geometry>
+  </collision>
+  <inertial>
+    <origin xyz="0 0 0" rpy="0 0 0"/>
+    <mass value="0.1"/>
+    <inertia ixx="0.001876" ixy="-0.001122" ixz="0.000392" iyy="0.004166" iyz="0.000374" izz="0.005261"/>
+  </inertial>
+</link>
+<link name="greifer_finger_2">
+  <visual>
+    <geometry>
+      <mesh filename="package://kr3r540_description/meshes/visual/Finger_2_visual.stl" scale="0.001 0.001 0.001"/>
+    </geometry>
+    <material name="kuka_pedestal">
+      <color rgba="0.50588 0.47059 0.38824 1.0"/>
+    </material>
+  </visual>
+  <collision>
+    <geometry>
+      <mesh filename="package://kr3r540_description/meshes/collision/Finger_2_collusion.stl" scale="0.001 0.001 0.001"/>
+    </geometry>
+  </collision>
+  <inertial>
+    <origin xyz="0 0 0" rpy="0 0 0"/>
+    <mass value="0.1"/>
+    <inertia ixx="0.001030" ixy="0.000654" ixz="0.000219" iyy="0.002527" iyz="-0.000204" izz="0.003130"/>
+  </inertial>
+</link>
+<!--
+<link name="greifer">
+  <visual>
+    <geometry>
+      <mesh filename="package://kr3r540_description/meshes/visual/greifer.stl" scale="0.1 0.1 0.1"/>
+    </geometry>
+    <material name="kuka_black">
+      <color rgba="0.0549 0.0549 0.0627 1.0"/>
+    </material>
+  </visual>
+  <collision>
+    <geometry>
       <mesh filename="package://kr3r540_description/meshes/collision/greifer.stl" scale="0.1 0.1 0.1"/>
     </geometry>
@@ -169,4 +231,5 @@
   </inertial>
 </link>
+-->
 <!-- Define Joints -->
 <joint name="world_to_base" type="fixed">
@@ -219,6 +282,20 @@
 <joint name="flange" type="fixed">
   <parent link="link_6"/>
-  <child link="greifer"/>
-  <origin xyz="0.032 0 0.02" rpy="0 ${2*1.5708} 1.5708"/>
+  <child link="greifer_base"/>
+  <origin xyz="0.013 0 0.02" rpy="1.57 ${-2*1.5708} -1.57"/>
+</joint>
+<joint name="flange_finger_1" type="prismatic">
+  <parent link="greifer_base"/>
+  <child link="greifer_finger_1"/>
+  <origin xyz="0 0 0" rpy="0 0 0"/>
+  <axis xyz="1 0 0"/>
+  <limit lower="0" upper="0.006" effort="10" velocity="0.1"/>
+</joint>
+<joint name="flange_finger_2" type="prismatic">
+  <parent link="greifer_base"/>
+  <child link="greifer_finger_2"/>
+  <origin xyz="0 0 0" rpy="0 0 0"/>
+  <axis xyz="-1 0 0"/>
+  <limit lower="0" upper="0.006" effort="10" velocity="0.1"/>
 </joint>
 </robot>

File: Software/ROS2_Env/kr3r540_ws/src/kr3r540_description/urdf/kr3r540_ros2_control.xacro (robot description, xacro)
@@ -58,4 +58,14 @@
             </state_interface>
         </joint>
+        <joint name="flange_finger_1">
+            <command_interface name="position">
+            </command_interface>
+            <state_interface name="position"/>
+        </joint>
+        <joint name="flange_finger_2">
+            <command_interface name="position">
+            </command_interface>
+            <state_interface name="position"/>
+        </joint>
     </ros2_control>
 </robot>

Commit message: Update : System now works with a gripper (fixed the gripper bugs)

File: Software/ROS2_Env/kr3r540_ws/src/kr3r540_description/urdf/kr3r540.urdf.xacro (robot description, xacro)
@@ -186,5 +186,5 @@
   <inertial>
     <origin xyz="0 0 0" rpy="0 0 0"/>
-    <mass value="0.1"/>
+    <mass value="0.01"/>
     <inertia ixx="0.001876" ixy="-0.001122" ixz="0.000392" iyy="0.004166" iyz="0.000374" izz="0.005261"/>
   </inertial>
@@ -206,5 +206,5 @@
   <inertial>
     <origin xyz="0 0 0" rpy="0 0 0"/>
-    <mass value="0.1"/>
+    <mass value="0.01"/>
     <inertia ixx="0.001030" ixy="0.000654" ixz="0.000219" iyy="0.002527" iyz="-0.000204" izz="0.003130"/>
   </inertial>
@@ -290,5 +290,5 @@
   <origin xyz="0 0 0" rpy="0 0 0"/>
   <axis xyz="1 0 0"/>
-  <limit lower="0" upper="0.006" effort="10" velocity="0.1"/>
+  <limit lower="0" upper="0.006" effort="100" velocity="0.1"/>
 </joint>
 <joint name="flange_finger_2" type="prismatic">
@@ -297,5 +297,5 @@
   <origin xyz="0 0 0" rpy="0 0 0"/>
   <axis xyz="-1 0 0"/>
-  <limit lower="0" upper="0.006" effort="10" velocity="0.1"/>
+  <limit lower="0" upper="0.006" effort="100" velocity="0.1"/>
 </joint>
 </robot>

File: Software/ROS2_Env/kr3r540_ws/src/kr3r540_description/urdf/kr3r540_ros2_control.xacro (robot description, xacro)
@@ -61,10 +61,14 @@
             <command_interface name="position">
             </command_interface>
-            <state_interface name="position"/>
+            <state_interface name="position">
+                <param name="initial_value">${initial_positions.initial_positions.flange_finger_1}</param>
+            </state_interface>
         </joint>
         <joint name="flange_finger_2">
             <command_interface name="position">
             </command_interface>
-            <state_interface name="position"/>
+            <state_interface name="position">
+                <param name="initial_value">${initial_positions.initial_positions.flange_finger_2}</param>
+            </state_interface>
         </joint>
     </ros2_control>
